Commit message: Fix namespace parameter in origin_one URDF xacro
Add missing xacro arg and property definitions for 'ns' variable used in IMU and camera frame IDs

Co-Authored-By: Claude Haiku 4.5 <noreply@anthropic.com>

File: origin_one_description/urdf/origin_one.urdf.xacro (robot description, xacro)
@@ -2,5 +2,7 @@
 <robot name="avular_origin_one" xmlns:xacro="http://ros.org/wiki/xacro" xmlns:ignition="http://sdformat.org/schemas/root.xsd">
   <xacro:arg name="drive_configuration" default="skid_steer_drive"/>
+  <xacro:arg name="ns" default="robot"/>
   <xacro:property name="var" value="$(arg drive_configuration)"/>
+  <xacro:property name="ns" value="$(arg ns)"/>
   <xacro:if value="${var == 'skid_steer_drive'}">
     <xacro:property name="trackWidth" value="0.500"/>
@@ -416,5 +418,5 @@
       <gz_frame_id>camera_link</gz_frame_id>
       <topic>/robot/camera</topic>
-      <update_rate>6</update_rate>
+      <update_rate>30</update_rate>
       <camera name="camera">
         <horizontal_fov>1.0472</horizontal_fov>
@@ -422,10 +424,10 @@
           <intrinsics>
             <!-- fx = fy = width / ( 2 * tan (hfov / 2 ) ) -->
-            <fx>554.25469</fx>
-            <fy>554.25469</fy>
+            <fx>1108.50938</fx>
+            <fy>1108.50938</fy>
             <!-- cx = ( width + 1 ) / 2 -->
-            <cx>320.5</cx>
+            <cx>640.5</cx>
             <!-- cy = ( height + 1 ) / 2 -->
-            <cy>240.5</cy>
+            <cy>480.5</cy>
             <s>0</s>
           </intrinsics>
@@ -440,6 +442,6 @@
         </distortion>
         <image>
-          <width>640</width>
-          <height>480</height>
+          <width>1280</width>
+          <height>960</height>
           <format>R8G8B8</format>
         </image>
@@ -514,4 +516,28 @@
   <link name="imu_link">
   </link>
+  <gazebo reference="imu_link">
+    <sensor name="imu_sensor" type="imu">
+      <gz_frame_id>${ns}/imu_link</gz_frame_id>
+      <always_on>1</always_on>
+      <update_rate>100</update_rate>
+      <topic>/model/${ns}/imu</topic>
+      <visualize>false</visualize>
+      <imu>
+        <orientation_reference_frame>
+          <localization>ENU</localization>
+        </orientation_reference_frame>
+        <angular_velocity>
+          <x><noise type="gaussian"><mean>0.0</mean><stddev>0.0002</stddev></noise></x>
+          <y><noise type="gaussian"><mean>0.0</mean><stddev>0.0002</stddev></noise></y>
+          <z><noise type="gaussian"><mean>0.0</mean><stddev>0.0002</stddev></noise></z>
+        </angular_velocity>
+        <linear_acceleration>
+          <x><noise type="gaussian"><mean>0.0</mean><stddev>0.017</stddev></noise></x>
+          <y><noise type="gaussian"><mean>0.0</mean><stddev>0.017</stddev></noise></y>
+          <z><noise type="gaussian"><mean>0.0</mean><stddev>0.017</stddev></noise></z>
+        </linear_acceleration>
+      </imu>
+    </sensor>
+  </gazebo>
   <joint type="fixed" name="base_body">
     <origin xyz="0.0 0 ${groundClearance}" rpy="0 0 0"/>
