Commit message: namespacing + unify sensors + avoid robot drifting on its own

File: origin_one_description/urdf/origin_one.urdf.xacro (robot description, xacro)
@@ -2,5 +2,7 @@
 <robot name="avular_origin_one" xmlns:xacro="http://ros.org/wiki/xacro" xmlns:ignition="http://sdformat.org/schemas/root.xsd">
   <xacro:arg name="drive_configuration" default="skid_steer_drive"/>
+  <xacro:arg name="robot_namespace" default="robot"/>
   <xacro:property name="var" value="$(arg drive_configuration)"/>
+  <xacro:property name="ns" value="$(arg robot_namespace)"/>
   <xacro:if value="${var == 'skid_steer_drive'}">
     <xacro:property name="trackWidth" value="0.500"/>
@@ -45,9 +47,5 @@
   <gazebo>
     <static>false</static>
-    <plugin filename="gz-sim-sensors-system" name="gz::sim::systems::Sensors">
-      <render_engine>ogre2</render_engine>
-    </plugin>
-    <plugin filename="ignition-gazebo-navsat-system" name="ignition::gazebo::systems::NavSat">
-    </plugin>
+    <!-- Sensors & NavSat system plugins are loaded at world level (baylands.world) -->
   </gazebo>
   <link name='base_link' />
@@ -98,5 +96,5 @@
               <mu>1</mu>
               <mu2>1</mu2>
-              <slip1>0.015</slip1>
+              <slip1>0.001</slip1>
               <slip2>0</slip2>
               <fdir1>0 0 1</fdir1>
@@ -114,5 +112,5 @@
               <mu>1</mu>
               <mu2>1</mu2>
-              <slip1>0.015</slip1>
+              <slip1>0.001</slip1>
               <slip2>0</slip2>
               <fdir1>0 0 1</fdir1>
@@ -123,5 +121,5 @@
               <mu>1</mu>
               <mu2>1</mu2>
-              <slip1>0.015</slip1>
+              <slip1>0.001</slip1>
               <slip2>0</slip2>
               <fdir1>0 0 1</fdir1>
@@ -164,5 +162,5 @@
               <mu>1</mu>
               <mu2>1</mu2>
-              <slip1>0.015</slip1>
+              <slip1>0.001</slip1>
               <slip2>0</slip2>
               <fdir1>0 0 1</fdir1>
@@ -180,5 +178,5 @@
               <mu>1</mu>
               <mu2>1</mu2>
-              <slip1>0.015</slip1>
+              <slip1>0.001</slip1>
               <slip2>0</slip2>
               <fdir1>0 0 1</fdir1>
@@ -189,5 +187,5 @@
               <mu>1</mu>
               <mu2>1</mu2>
-              <slip1>0.015</slip1>
+              <slip1>0.001</slip1>
               <slip2>0</slip2>
               <fdir1>0 0 1</fdir1>
@@ -230,5 +228,5 @@
               <mu>1</mu>
               <mu2>1</mu2>
-              <slip1>0.015</slip1>
+              <slip1>0.001</slip1>
               <slip2>0</slip2>
               <fdir1>0 0 1</fdir1>
@@ -246,5 +244,5 @@
               <mu>1</mu>
               <mu2>1</mu2>
-              <slip1>0.015</slip1>
+              <slip1>0.001</slip1>
               <slip2>0</slip2>
               <fdir1>0 0 1</fdir1>
@@ -255,5 +253,5 @@
               <mu>1</mu>
               <mu2>1</mu2>
-              <slip1>0.015</slip1>
+              <slip1>0.001</slip1>
               <slip2>0</slip2>
               <fdir1>0 0 1</fdir1>
@@ -296,5 +294,5 @@
               <mu>1</mu>
               <mu2>1</mu2>
-              <slip1>0.015</slip1>
+              <slip1>0.001</slip1>
               <slip2>0</slip2>
               <fdir1>0 0 1</fdir1>
@@ -312,5 +310,5 @@
               <mu>1</mu>
               <mu2>1</mu2>
-              <slip1>0.015</slip1>
+              <slip1>0.001</slip1>
               <slip2>0</slip2>
               <fdir1>0 0 1</fdir1>
@@ -321,5 +319,5 @@
               <mu>1</mu>
               <mu2>1</mu2>
-              <slip1>0.015</slip1>
+              <slip1>0.001</slip1>
               <slip2>0</slip2>
               <fdir1>0 0 1</fdir1>
@@ -368,6 +366,6 @@
   <gazebo reference="lidar_link_gazebo">
     <sensor name='ouster_lidar' type='gpu_lidar'>
-      <topic>/robot/lidar</topic>
-      <gz_frame_id>os_lidar</gz_frame_id>
+      <topic>/model/${ns}/lidar</topic>
+      <gz_frame_id>${ns}/lidar_link_gazebo</gz_frame_id>
       <update_rate>10</update_rate>
       <lidar>
@@ -414,6 +412,6 @@
   <gazebo reference="camera_link">
     <sensor name="realsense_d435" type="rgbd_camera">
-      <gz_frame_id>camera_link</gz_frame_id>
-      <topic>/robot/camera</topic>
+      <gz_frame_id>${ns}/camera_link</gz_frame_id>
+      <topic>/model/${ns}/camera</topic>
       <update_rate>6</update_rate>
       <camera name="camera">
@@ -475,8 +473,8 @@
   <gazebo reference="gnss_link">
     <sensor name="navsat" type="navsat">
-      <gz_frame_id>gnss_link</gz_frame_id>
+      <gz_frame_id>${ns}/gnss_link</gz_frame_id>
       <always_on>1</always_on>
       <update_rate>10</update_rate>
-      <topic>/robot/gnss</topic>
+      <topic>/model/${ns}/navsat</topic>
       <!-- Obtained from http://sdformat.org/spec?ver=1.11&elem=sensor#sensor_gps -->
       <gps>
@@ -525,4 +523,5 @@
     <axis xyz="0 0 1"/>
     <limit effort="100000.0" velocity="10"/>
+    <dynamics damping="0.5" friction="0.3"/>
   </joint>
   <joint type="continuous" name="main_body_right_front_wheel">
@@ -532,4 +531,5 @@
     <axis xyz="0 0 1"/>
     <limit effort="100000.0" velocity="10"/>
+    <dynamics damping="0.5" friction="0.3"/>
   </joint>
   <joint type="continuous" name="main_body_left_rear_wheel">
@@ -539,4 +539,5 @@
     <axis xyz="0 0 1"/>
     <limit effort="100000.0" velocity="10"/>
+    <dynamics damping="0.5" friction="0.3"/>
   </joint>
   <joint type="continuous" name="main_body_right_rear_wheel">
@@ -546,4 +547,5 @@
     <axis xyz="0 0 1"/>
     <limit effort="100000.0" velocity="10"/>
+    <dynamics damping="0.5" friction="0.3"/>
   </joint>
   <joint type="fixed" name="ouster_platform_joint">
@@ -609,5 +611,5 @@
   <gazebo>
     <plugin filename="gz-sim-joint-state-publisher-system" name="ignition::gazebo::systems::JointStatePublisher">
-      <topic>/robot/joint_states</topic>
+      <topic>/model/${ns}/joint_state</topic>
     </plugin>
     <!-- Controls the differential drive robot -->
@@ -628,9 +630,9 @@
         <max_angular_velocity>2</max_angular_velocity>
         <min_angular_velocity>-2</min_angular_velocity>
-        <topic>/robot/cmd_vel</topic>
-        <odom_topic>/robot/odom</odom_topic>
-        <tf_topic>/robot/tf</tf_topic>
-        <frame_id>odom</frame_id>
-        <child_frame_id>base_link</child_frame_id>
+        <topic>/model/${ns}/cmd_vel</topic>
+        <odom_topic>/model/${ns}/odometry</odom_topic>
+        <tf_topic>/model/${ns}/tf</tf_topic>
+        <frame_id>${ns}/odom</frame_id>
+        <child_frame_id>${ns}/base_link</child_frame_id>
       </plugin>
     </xacro:if>
@@ -652,9 +654,9 @@
         <max_angular_velocity>3</max_angular_velocity>
         <min_angular_velocity>-3</min_angular_velocity>
-        <topic>/robot/cmd_vel</topic>
-        <odom_topic>/robot/odom</odom_topic>
-        <tf_topic>/robot/tf</tf_topic>
-        <frame_id>odom</frame_id>
-        <child_frame_id>base_link</child_frame_id>
+        <topic>/model/${ns}/cmd_vel</topic>
+        <odom_topic>/model/${ns}/odometry</odom_topic>
+        <tf_topic>/model/${ns}/tf</tf_topic>
+        <frame_id>${ns}/odom</frame_id>
+        <child_frame_id>${ns}/base_link</child_frame_id>
       </plugin>
     </xacro:if>
@@ -676,9 +678,9 @@
         <max_angular_velocity>3</max_angular_velocity>
         <min_angular_velocity>-3</min_angular_velocity>
-        <topic>/robot/cmd_vel</topic>
-        <odom_topic>/robot/odom</odom_topic>
-        <tf_topic>/robot/tf</tf_topic>
-        <frame_id>odom</frame_id>
-        <child_frame_id>base_link</child_frame_id>
+        <topic>/model/${ns}/cmd_vel</topic>
+        <odom_topic>/model/${ns}/odometry</odom_topic>
+        <tf_topic>/model/${ns}/tf</tf_topic>
+        <frame_id>${ns}/odom</frame_id>
+        <child_frame_id>${ns}/base_link</child_frame_id>
       </plugin>
     </xacro:if>
@@ -696,5 +698,5 @@
         <min_acceleration>-5</min_acceleration>
         <max_acceleration>5</max_acceleration>
-        <topic>/robot/cmd_vel</topic>
+        <topic>/model/${ns}/cmd_vel</topic>
       </plugin>
     <!-- Seperate plugin for odometry is used because mecanum drive plug does not have this feature-->
@@ -702,8 +704,8 @@
       <plugin
         filename="gz-sim-odometry-publisher-system" name="ignition::gazebo::systems::OdometryPublisher">
-        <odom_topic>/robot/odom</odom_topic>
-        <tf_topic>/robot/tf</tf_topic>
-        <odom_frame>odom</odom_frame>
-        <robot_base_frame>base_link</robot_base_frame>
+        <odom_topic>/model/${ns}/odometry</odom_topic>
+        <tf_topic>/model/${ns}/tf</tf_topic>
+        <odom_frame>${ns}/odom</odom_frame>
+        <robot_base_frame>${ns}/base_link</robot_base_frame>
       </plugin>
     </xacro:if>

Commit message: fix imu orientation

File: origin_one_description/urdf/origin_one.urdf.xacro (robot description, xacro)
@@ -512,4 +512,25 @@
   <link name="imu_link">
   </link>
+  <gazebo reference="imu_link">
+    <sensor name="imu_sensor" type="imu">
+      <gz_frame_id>${ns}/imu_link</gz_frame_id>
+      <always_on>1</always_on>
+      <update_rate>100</update_rate>
+      <topic>/model/${ns}/imu</topic>
+      <visualize>false</visualize>
+      <imu>
+        <angular_velocity>
+          <x><noise type="gaussian"><mean>0.0</mean><stddev>0.0002</stddev></noise></x>
+          <y><noise type="gaussian"><mean>0.0</mean><stddev>0.0002</stddev></noise></y>
+          <z><noise type="gaussian"><mean>0.0</mean><stddev>0.0002</stddev></noise></z>
+        </angular_velocity>
+        <linear_acceleration>
+          <x><noise type="gaussian"><mean>0.0</mean><stddev>0.017</stddev></noise></x>
+          <y><noise type="gaussian"><mean>0.0</mean><stddev>0.017</stddev></noise></y>
+          <z><noise type="gaussian"><mean>0.0</mean><stddev>0.017</stddev></noise></z>
+        </linear_acceleration>
+      </imu>
+    </sensor>
+  </gazebo>
   <joint type="fixed" name="base_body">
     <origin xyz="0.0 0 ${groundClearance}" rpy="0 0 0"/>
@@ -605,5 +626,5 @@
   </joint>
   <joint type="fixed" name="imu_joint">
-    <origin xyz="-0.1266 0.0749 0.066" rpy="0 0 2.357"/>
+    <origin xyz="-0.1266 0.0749 0.066" rpy="0 0 0"/>
     <child link="imu_link"/>
     <parent link="main_body"/>

Commit message: fix stuff?

File: origin_one_description/urdf/origin_one.urdf.xacro (robot description, xacro)
@@ -2,7 +2,7 @@
 <robot name="avular_origin_one" xmlns:xacro="http://ros.org/wiki/xacro" xmlns:ignition="http://sdformat.org/schemas/root.xsd">
   <xacro:arg name="drive_configuration" default="skid_steer_drive"/>
-  <xacro:arg name="ns" default="robot"/>
+  <xacro:arg name="robot_namespace" default="robot"/>
   <xacro:property name="var" value="$(arg drive_configuration)"/>
-  <xacro:property name="ns" value="$(arg ns)"/>
+  <xacro:property name="ns" value="$(arg robot_namespace)"/>
   <xacro:if value="${var == 'skid_steer_drive'}">
     <xacro:property name="trackWidth" value="0.500"/>
@@ -47,9 +47,5 @@
   <gazebo>
     <static>false</static>
-    <plugin filename="ignition-gazebo-navsat-system" name="ignition::gazebo::systems::NavSat">
-    </plugin>
-    <plugin filename="gz-sim-sensors-system" name="gz::sim::systems::Sensors">
-      <render_engine>ogre2</render_engine>
-    </plugin>
+    <!-- Sensors & NavSat system plugins are loaded at world level (baylands.world) -->
   </gazebo>
   <link name='base_link' />
@@ -100,5 +96,5 @@
               <mu>1</mu>
               <mu2>1</mu2>
-              <slip1>0.015</slip1>
+              <slip1>0.001</slip1>
               <slip2>0</slip2>
               <fdir1>0 0 1</fdir1>
@@ -116,5 +112,5 @@
               <mu>1</mu>
               <mu2>1</mu2>
-              <slip1>0.015</slip1>
+              <slip1>0.001</slip1>
               <slip2>0</slip2>
               <fdir1>0 0 1</fdir1>
@@ -125,5 +121,5 @@
               <mu>1</mu>
               <mu2>1</mu2>
-              <slip1>0.015</slip1>
+              <slip1>0.001</slip1>
               <slip2>0</slip2>
               <fdir1>0 0 1</fdir1>
@@ -166,5 +162,5 @@
               <mu>1</mu>
               <mu2>1</mu2>
-              <slip1>0.015</slip1>
+              <slip1>0.001</slip1>
               <slip2>0</slip2>
               <fdir1>0 0 1</fdir1>
@@ -182,5 +178,5 @@
               <mu>1</mu>
               <mu2>1</mu2>
-              <slip1>0.015</slip1>
+              <slip1>0.001</slip1>
               <slip2>0</slip2>
               <fdir1>0 0 1</fdir1>
@@ -191,5 +187,5 @@
               <mu>1</mu>
               <mu2>1</mu2>
-              <slip1>0.015</slip1>
+              <slip1>0.001</slip1>
               <slip2>0</slip2>
               <fdir1>0 0 1</fdir1>
@@ -232,5 +228,5 @@
               <mu>1</mu>
               <mu2>1</mu2>
-              <slip1>0.015</slip1>
+              <slip1>0.001</slip1>
               <slip2>0</slip2>
               <fdir1>0 0 1</fdir1>
@@ -248,5 +244,5 @@
               <mu>1</mu>
               <mu2>1</mu2>
-              <slip1>0.015</slip1>
+              <slip1>0.001</slip1>
               <slip2>0</slip2>
               <fdir1>0 0 1</fdir1>
@@ -257,5 +253,5 @@
               <mu>1</mu>
               <mu2>1</mu2>
-              <slip1>0.015</slip1>
+              <slip1>0.001</slip1>
               <slip2>0</slip2>
               <fdir1>0 0 1</fdir1>
@@ -298,5 +294,5 @@
               <mu>1</mu>
               <mu2>1</mu2>
-              <slip1>0.015</slip1>
+              <slip1>0.001</slip1>
               <slip2>0</slip2>
               <fdir1>0 0 1</fdir1>
@@ -314,5 +310,5 @@
               <mu>1</mu>
               <mu2>1</mu2>
-              <slip1>0.015</slip1>
+              <slip1>0.001</slip1>
               <slip2>0</slip2>
               <fdir1>0 0 1</fdir1>
@@ -323,5 +319,5 @@
               <mu>1</mu>
               <mu2>1</mu2>
-              <slip1>0.015</slip1>
+              <slip1>0.001</slip1>
               <slip2>0</slip2>
               <fdir1>0 0 1</fdir1>
@@ -370,6 +366,6 @@
   <gazebo reference="lidar_link_gazebo">
     <sensor name='ouster_lidar' type='gpu_lidar'>
-      <topic>/robot/lidar</topic>
-      <gz_frame_id>os_lidar</gz_frame_id>
+      <topic>/model/${ns}/lidar</topic>
+      <gz_frame_id>${ns}/lidar_link_gazebo</gz_frame_id>
       <update_rate>10</update_rate>
       <lidar>
@@ -416,7 +412,7 @@
   <gazebo reference="camera_link">
     <sensor name="realsense_d435" type="rgbd_camera">
-      <gz_frame_id>camera_link</gz_frame_id>
-      <topic>/robot/camera</topic>
-      <update_rate>30</update_rate>
+      <gz_frame_id>${ns}/camera_link</gz_frame_id>
+      <topic>/model/${ns}/camera</topic>
+      <update_rate>6</update_rate>
       <camera name="camera">
         <horizontal_fov>1.0472</horizontal_fov>
@@ -477,8 +473,8 @@
   <gazebo reference="gnss_link">
     <sensor name="navsat" type="navsat">
-      <gz_frame_id>gnss_link</gz_frame_id>
+      <gz_frame_id>${ns}/gnss_link</gz_frame_id>
       <always_on>1</always_on>
       <update_rate>10</update_rate>
-      <topic>/robot/gnss</topic>
+      <topic>/model/${ns}/navsat</topic>
       <!-- Obtained from http://sdformat.org/spec?ver=1.11&elem=sensor#sensor_gps -->
       <gps>
@@ -488,5 +484,5 @@
             <noise type="gaussian">
               <mean>0.0</mean>
-              <stddev>0.0001</stddev>
+              <stddev>0.000</stddev>
             </noise>
           </horizontal>
@@ -524,7 +520,4 @@
       <visualize>false</visualize>
       <imu>
-        <orientation_reference_frame>
-          <localization>ENU</localization>
-        </orientation_reference_frame>
         <angular_velocity>
           <x><noise type="gaussian"><mean>0.0</mean><stddev>0.0002</stddev></noise></x>
@@ -551,4 +544,5 @@
     <axis xyz="0 0 1"/>
     <limit effort="100000.0" velocity="10"/>
+    <dynamics damping="0.5" friction="0.3"/>
   </joint>
   <joint type="continuous" name="main_body_right_front_wheel">
@@ -558,4 +552,5 @@
     <axis xyz="0 0 1"/>
     <limit effort="100000.0" velocity="10"/>
+    <dynamics damping="0.5" friction="0.3"/>
   </joint>
   <joint type="continuous" name="main_body_left_rear_wheel">
@@ -565,4 +560,5 @@
     <axis xyz="0 0 1"/>
     <limit effort="100000.0" velocity="10"/>
+    <dynamics damping="0.5" friction="0.3"/>
   </joint>
   <joint type="continuous" name="main_body_right_rear_wheel">
@@ -572,4 +568,5 @@
     <axis xyz="0 0 1"/>
     <limit effort="100000.0" velocity="10"/>
+    <dynamics damping="0.5" friction="0.3"/>
   </joint>
   <joint type="fixed" name="ouster_platform_joint">
@@ -629,5 +626,5 @@
   </joint>
   <joint type="fixed" name="imu_joint">
-    <origin xyz="-0.1266 0.0749 0.066" rpy="0 0 2.357"/>
+    <origin xyz="-0.1266 0.0749 0.066" rpy="0 0 0"/>
     <child link="imu_link"/>
     <parent link="main_body"/>
@@ -635,5 +632,5 @@
   <gazebo>
     <plugin filename="gz-sim-joint-state-publisher-system" name="ignition::gazebo::systems::JointStatePublisher">
-      <topic>/robot/joint_states</topic>
+      <topic>/model/${ns}/joint_state</topic>
     </plugin>
     <!-- Controls the differential drive robot -->
@@ -654,9 +651,9 @@
         <max_angular_velocity>2</max_angular_velocity>
         <min_angular_velocity>-2</min_angular_velocity>
-        <topic>/robot/cmd_vel</topic>
-        <odom_topic>/robot/odom</odom_topic>
-        <tf_topic>/robot/tf</tf_topic>
-        <frame_id>odom</frame_id>
-        <child_frame_id>base_link</child_frame_id>
+        <topic>/model/${ns}/cmd_vel</topic>
+        <odom_topic>/model/${ns}/odometry</odom_topic>
+        <tf_topic>/model/${ns}/tf</tf_topic>
+        <frame_id>${ns}/odom</frame_id>
+        <child_frame_id>${ns}/base_link</child_frame_id>
       </plugin>
     </xacro:if>
@@ -678,9 +675,9 @@
         <max_angular_velocity>3</max_angular_velocity>
         <min_angular_velocity>-3</min_angular_velocity>
-        <topic>/robot/cmd_vel</topic>
-        <odom_topic>/robot/odom</odom_topic>
-        <tf_topic>/robot/tf</tf_topic>
-        <frame_id>odom</frame_id>
-        <child_frame_id>base_link</child_frame_id>
+        <topic>/model/${ns}/cmd_vel</topic>
+        <odom_topic>/model/${ns}/odometry</odom_topic>
+        <tf_topic>/model/${ns}/tf</tf_topic>
+        <frame_id>${ns}/odom</frame_id>
+        <child_frame_id>${ns}/base_link</child_frame_id>
       </plugin>
     </xacro:if>
@@ -702,9 +699,9 @@
         <max_angular_velocity>3</max_angular_velocity>
         <min_angular_velocity>-3</min_angular_velocity>
-        <topic>/robot/cmd_vel</topic>
-        <odom_topic>/robot/odom</odom_topic>
-        <tf_topic>/robot/tf</tf_topic>
-        <frame_id>odom</frame_id>
-        <child_frame_id>base_link</child_frame_id>
+        <topic>/model/${ns}/cmd_vel</topic>
+        <odom_topic>/model/${ns}/odometry</odom_topic>
+        <tf_topic>/model/${ns}/tf</tf_topic>
+        <frame_id>${ns}/odom</frame_id>
+        <child_frame_id>${ns}/base_link</child_frame_id>
       </plugin>
     </xacro:if>
@@ -722,5 +719,5 @@
         <min_acceleration>-5</min_acceleration>
         <max_acceleration>5</max_acceleration>
-        <topic>/robot/cmd_vel</topic>
+        <topic>/model/${ns}/cmd_vel</topic>
       </plugin>
     <!-- Seperate plugin for odometry is used because mecanum drive plug does not have this feature-->
@@ -728,8 +725,8 @@
       <plugin
         filename="gz-sim-odometry-publisher-system" name="ignition::gazebo::systems::OdometryPublisher">
-        <odom_topic>/robot/odom</odom_topic>
-        <tf_topic>/robot/tf</tf_topic>
-        <odom_frame>odom</odom_frame>
-        <robot_base_frame>base_link</robot_base_frame>
+        <odom_topic>/model/${ns}/odometry</odom_topic>
+        <tf_topic>/model/${ns}/tf</tf_topic>
+        <odom_frame>${ns}/odom</odom_frame>
+        <robot_base_frame>${ns}/base_link</robot_base_frame>
       </plugin>
     </xacro:if>
